File: Arm_stepper.kicad_pcb (KiCad board)
At the start: 2 copper layers, 134 parts, among them IC1 L6208D, IC2 L6208D, J1 12V_CONN, J10 ENCODER1, J11 ENCODER2, J2 M1_CONN, J3 M1_CONN, J4 Conn_01x06_Male, J5 I2C_CONN, J8 Conn_01x04_Female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

Commit message: mcu circuitry drawn
Parts:
- removed D7: 1N4148, Diodes_SMD:D_SOD-123
- added C13: 220nF1, Capacitors_SMD:C_1206_HandSoldering, F.Cu at (325.0, 88.4)
- added C17: 10nF, Capacitors_SMD:C_1206_HandSoldering, F.Cu at (325.0, 99.8)
- added C21: 100nF, Capacitors_SMD:C_1206_HandSoldering, F.Cu at (357.1, 65.4)
- added C22: 100uF ceramic, Capacitors_SMD:C_1206_HandSoldering, F.Cu at (360.9, 65.4)
- added C23: 1nF, Capacitors_SMD:C_1206_HandSoldering, F.Cu at (375.2, 84.0)
- added C24: 1nF, Capacitors_SMD:C_1206_HandSoldering, F.Cu at (342.1, 84.0)
- added C28: 68nF, Capacitors_SMD:C_1206_HandSoldering, F.Cu at (380.0, 102.2)
- added C3: 5.6n, Capacitors_SMD:C_1206_HandSoldering, F.Cu at (340.2, 96.1)
- added C30: 68nF, Capacitors_SMD:C_1206_HandSoldering, F.Cu at (340.2, 102.4)
- added C7: 100nF, Capacitors_SMD:C_1206_HandSoldering, F.Cu at (377.9, 97.6)
- added D1: 1N4148, Diodes_SMD:D_1206, F.Cu at (321.8, 92.8)
- added D15: LED, LEDs:LED_1206_HandSoldering, F.Cu at (370.3, 112.6)
- added D16: LED, LEDs:LED_1206_HandSoldering, F.Cu at (339.1, 115.4)
- added D17: LED, LEDs:LED_1206_HandSoldering, F.Cu at (378.0, 116.0)
- added D18: LED, LEDs:LED_1206_HandSoldering, F.Cu at (332.0, 115.4)
- added D5: 1N4148, Diodes_SMD:D_SOD-123, F.Cu at (328.2, 92.8)
- added HS1: Heatsink_Pad, SMD_Packages:1Pin, F.Cu at (361.1, 74.1)
- added HS1: Heatsink_Pad, SMD_Packages:1Pin, F.Cu at (363.1, 103.3)
- added IC1: L6208D, Arm_stepper:POWERSO36, F.Cu at (358.6, 90.3)
- added J3: M1_CONN, TerminalBlocks_Phoenix:TerminalBlock_Phoenix_PT-3.5mm_4pol, F.Cu at (353.6, 114.4)
- added JP4: SolderJumper_2_Bridged, Wire_Connections_Bridges:WireConnection_1.50mmDrill, F.Cu at (319.0, 68.7)
- added R10: 100, Resistors_SMD:R_1206_HandSoldering, F.Cu at (332.0, 97.9)
- added R12: 39k, Resistors_SMD:R_1206_HandSoldering, F.Cu at (372.0, 83.9)
- added R13: 39k, Resistors_SMD:R_1206_HandSoldering, F.Cu at (339.0, 83.9)
- added R14: 0.3, Resistors_SMD:R_2512_HandSoldering, F.Cu at (380.2, 85.0)
- added R17: 0.3, Resistors_SMD:R_2512_HandSoldering, F.Cu at (333.9, 84.6)
- added R19: 2.2K, Resistors_SMD:R_1206_HandSoldering, F.Cu at (380.0, 105.5)
- added R25: 2.2K, Resistors_SMD:R_1206_HandSoldering, F.Cu at (340.1, 105.5)
- added R34: 4.7K, Resistors_SMD:R_1206_HandSoldering, F.Cu at (378.0, 110.6)
- added R35: 4.7K, Resistors_SMD:R_1206_HandSoldering, F.Cu at (342.1, 110.6)
- added R4: 100k, Resistors_SMD:R_1206_HandSoldering, F.Cu at (340.1, 99.2)
- added R41: 10K, Resistors_SMD:R_1206_HandSoldering, F.Cu at (370.3, 115.2)
- added R42: 10K, Resistors_SMD:R_1206_HandSoldering, F.Cu at (339.1, 118.2)
- added R43: 10K, Resistors_SMD:R_1206_HandSoldering, F.Cu at (370.3, 118.0)
- added R44: 10K, Resistors_SMD:R_1206_HandSoldering, F.Cu at (332.0, 118.2)
- SW1: footprint SMD_Packages:1Pin -> Buttons_Switches_THT:SW_TH_Tactile_Omron_B3F-10xx
- moved J11 170.2 mm to (135.6, 114.7)
- moved D9 168.1 mm to (147.6, 106.9), turned to 90 degrees
- moved C6 165.6 mm to (162.8, 107.0), turned to 90 degrees
- moved SW3 164.7 mm to (147.1, 114.6)
- moved R21 163.8 mm to (150.2, 106.9), turned to 90 degrees
- moved SW5 160.2 mm to (165.7, 114.6)
- moved C9 159.4 mm to (139.2, 104.1), turned to 315 degrees
- moved R48 156.0 mm to (145.2, 102.5), turned to 45 degrees
- moved J10 155.6 mm to (124.1, 114.7)
- moved SW1 153.4 mm to (130.6, 91.3), turned to 45 degrees
- moved C34 153.0 mm to (140.6, 69.3), turned to 180 degrees
- moved SW2 151.3 mm to (153.3, 114.6)
- moved C8 147.6 mm to (143.1, 100.6), turned to 225 degrees
- moved Y1 144.4 mm to (134.0, 106.2), turned to 135 degrees
- moved U2 143.0 mm to (131.2, 82.8), turned to 270 degrees
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Connections:
- C13 pad 1: Net-(C13-Pad1) -> +12V
- C21 pad 1: Net-(C13-Pad1) -> +12V
- C22 pad 1: Net-(C13-Pad1) -> +12V
- D5 pad 2: Net-(C13-Pad1) -> +12V
- IC1 pad 33: Net-(C13-Pad1) -> +12V
- IC1 pad 4: Net-(C13-Pad1) -> +12V
- U3 pad 34: Net-(U3-Pad34) -> EN1
Routing:
- net +12V: track 60.2 -> 352.9 mm
- net GNDS: track 127.0 -> 280.3 mm, vias 16 -> 34
- net +3V3: track 0.00 -> 150.8 mm, vias 0 -> 26
- net Net-(C13-Pad1): track 149.0 -> 0.00 mm
- net E2: track 0.00 -> 77.2 mm
- net /M2_B-: track 68.1 -> 136.2 mm, vias 2 -> 4
- net /M2_A+: track 63.5 -> 127.1 mm, vias 2 -> 4
- net E1: track 0.00 -> 60.3 mm, vias 0 -> 4
- net /M2_B+: track 60.1 -> 120.2 mm, vias 2 -> 4
- net E4: track 0.00 -> 58.4 mm, vias 0 -> 1
- net /M2_A-: track 58.2 -> 116.5 mm
- net E3: track 0.00 -> 54.0 mm, vias 0 -> 2
- net Net-(C3-Pad1): track 38.7 -> 76.8 mm, vias 2 -> 4
- net Net-(C13-Pad2): track 36.9 -> 73.9 mm, vias 2 -> 4
- net +5V: track 0.00 -> 36.9 mm, vias 0 -> 14
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- added copper zone on B.Cu, net +3V3
- added copper zone on F.Cu, net +3V3

Commit message: pcb design almost complete
Parts:
- R24: value 1K -> 27K
- moved R7 145.5 mm to (158.2, 74.4), turned to 315 degrees
- moved TH1 138.5 mm to (191.6, 74.7), turned to 90 degrees
- moved Q2 131.1 mm to (177.5, 71.4)
- moved R46 126.0 mm to (141.0, 82.2), turned to 135 degrees
- moved C11 112.4 mm to (132.9, 70.5)
- moved R5 110.0 mm to (152.0, 74.2)
- moved R45 108.3 mm to (142.6, 80.4), turned to 315 degrees
- moved R31 105.6 mm to (175.3, 76.6), turned to 90 degrees
- moved M2 99.0 mm to (180.7, 67.7), turned to 90 degrees
- moved R24 94.7 mm to (186.9, 76.4)
- moved R6 91.3 mm to (152.0, 71.8)
- moved D2 29.9 mm to (145.7, 72.8)
- moved J5 8.89 mm to (125.1, 95.4)
- moved J9 6.22 mm to (124.6, 86.5)
- moved C14 2.47 mm to (137.7, 85.7)
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Connections:
- M1 pad 1: +5V -> +12V
- M2 pad 1: +5V -> +12V
- R24 pad 1: +3V3 -> +12V
- U3 pad 29: FAN -> Net-(U3-Pad29)
- U3 pad 4: Net-(U3-Pad4) -> FAN
Routing:
- net PWMA1: track 0.00 -> 110.4 mm, vias 0 -> 2
- net CRTL1: track 0.00 -> 107.2 mm, vias 0 -> 2
- net +5V: track 36.9 -> 121.3 mm, vias 14 -> 16
- net CLK1: track 0.00 -> 72.2 mm, vias 0 -> 2
- net RST1: track 37.3 -> 109.2 mm, vias 4 -> 5
- net GNDS: track 280.3 -> 348.8 mm, vias 34 -> 55
- net CW1: track 0.00 -> 67.3 mm, vias 0 -> 2
- net +3V3: track 150.8 -> 213.2 mm, vias 26 -> 34
- net EN1: track 0.00 -> 56.8 mm, vias 0 -> 4
- net PWMB1: track 0.00 -> 56.3 mm, vias 0 -> 2
- net t_SENS: track 0.00 -> 50.9 mm, vias 0 -> 2
- net HALF1: track 0.00 -> 49.7 mm, vias 0 -> 4
- net FAN: track 0.00 -> 44.1 mm, vias 0 -> 2
- net E2_2: track 0.00 -> 42.7 mm, vias 0 -> 2
- net E2_1: track 0.00 -> 40.5 mm, vias 0 -> 1
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
Commit message: copper completed
Parts:
- removed C15: 220nF1, Capacitors_SMD:C_1206_HandSoldering
- removed C18: 5.6n, Capacitors_SMD:C_1206_HandSoldering
- removed C19, C25, C6: 100nF, Capacitors_SMD:C_1206_HandSoldering
- removed C20: 10nF, Capacitors_SMD:C_1206_HandSoldering
- removed C29: 100uF ceramic, Capacitors_SMD:C_1206_HandSoldering
- removed C32, C33: 1nF, Capacitors_SMD:C_1206_HandSoldering
- removed C36, C38: 68nF, Capacitors_SMD:C_1206_HandSoldering
- removed D10: LED_RED, LEDs:LED_1206_HandSoldering
- removed D11, D12, D13, D14: LED, LEDs:LED_1206_HandSoldering
- removed D4, D6, D8: 1N4148, Diodes_SMD:D_SOD-123
- removed IC2: L6208D, Arm_stepper:POWERSO36
- removed J2: M1_CONN, TerminalBlocks_Phoenix:TerminalBlock_Phoenix_PT-3.5mm_4pol
- removed JP1, JP2, JP3: SolderJumper_2_Bridged, Pin_Headers:Pin_Header_Angled_1x03_Pitch2.54mm
- removed JP5: SolderJumper_2_Bridged, Wire_Connections_Bridges:WireConnection_1.50mmDrill
- removed L1: L, Inductors_SMD:L_1206_HandSoldering
- removed M1: Fan, Pin_Headers:Pin_Header_Angled_1x02_Pitch2.54mm
- removed Q1: 2N2219, TO_SOT_Packages_SMD:SOT-23
- removed R11: 100, Resistors_SMD:R_1206_HandSoldering
- removed R15, R16: 39k, Resistors_SMD:R_1206_HandSoldering
- removed R18, R20: 0.3, Resistors_SMD:R_2512_HandSoldering
- removed R22: 1k, Resistors_SMD:R_1206_HandSoldering
- removed R23, R36: 4.7K, Resistors_SMD:R_1206_HandSoldering
- removed R26, R33: 2.2K, Resistors_SMD:R_1206_HandSoldering
- removed R27: 70k, Resistors_SMD:R_1206_HandSoldering
- removed R37, R38, R39, R40: 10K, Resistors_SMD:R_1206_HandSoldering
- removed R9: 100k, Resistors_SMD:R_1206_HandSoldering
- added M2: Fan, Pin_Headers:Pin_Header_Angled_1x02_Pitch2.54mm, F.Cu at (177.4, 70.9)
- moved C35 198.5 mm to (94.9, 109.4), turned to 270 degrees
- moved JP4 171.6 mm to (147.4, 67.3)
- moved C21 154.1 mm to (203.0, 65.0)
- moved C22 154.1 mm to (206.8, 65.1)
- moved C23 154.1 mm to (221.0, 83.7)
- moved C7 154.1 mm to (223.8, 97.2)
- moved D18 154.1 mm to (177.9, 115.1)
- moved HS1 154.1 mm to (207.0, 73.8)
- moved HS1 154.1 mm to (209.0, 102.9)
- moved IC1 154.1 mm to (204.5, 89.9)
- moved R10 154.1 mm to (177.9, 97.5)
- moved R13 154.1 mm to (184.8, 83.6)
- moved R44 154.1 mm to (177.9, 117.9)
- moved C13 154.1 mm to (170.9, 88.0)
- moved C17 154.1 mm to (170.9, 99.4)
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Connections:
- R47 pad 1: Net-(R47-Pad1) -> /NRST
- U3 pad 12: GNDA -> GNDS
- U3 pad 13: Net-(JP2-Pad1) -> +3V3
- U3 pad 7: Net-(R47-Pad1) -> /NRST
Routing:
- net /NRST: track 0.00 -> 157.7 mm, vias 0 -> 3
- net CW1: track 67.3 -> 216.3 mm, vias 2 -> 5
- net HALF1: track 49.7 -> 186.3 mm, vias 4 -> 7
- net CLK1: track 72.2 -> 194.5 mm, vias 2 -> 5
- net CRTL1: track 107.2 -> 228.1 mm, vias 2 -> 3
- net Net-(C3-Pad1): track 76.8 -> 174.7 mm, vias 4 -> 6
- net GNDS: track 348.8 -> 432.0 mm, vias 55 -> 78
- net PWMA1: track 110.4 -> 182.2 mm, vias 2 -> 4
- net Net-(C30-Pad2): track 51.8 -> 123.3 mm, vias 4 -> 6
- net PWMB1: track 56.3 -> 126.9 mm, vias 2 -> 4
- net Net-(M2-Pad2): track 6.28 -> 75.8 mm
- net RST1: track 109.2 -> 167.1 mm, vias 5 -> 6
- net +12V: track 372.2 -> 429.1 mm
- net Net-(R5-Pad2): track 0.00 -> 48.3 mm, vias 0 -> 4
- net +3V3: track 213.2 -> 242.3 mm, vias 34 -> 35
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- added copper zone on B.Cu, net GNDD
Other:
- board outline added: 178.3 x 60.5 mm

Commit message: copper compl1
Parts:
- added REF**: MountingHole_3.2mm_M3, Mounting_Holes:MountingHole_3.2mm_M3, F.Cu at (226.8, 63.9)
- added REF**: MountingHole_3.2mm_M3, Mounting_Holes:MountingHole_3.2mm_M3, F.Cu at (229.1, 117.0)
- added REF**: MountingHole_3.2mm_M3, Mounting_Holes:MountingHole_3.2mm_M3, F.Cu at (57.8, 109.7)
- added REF**: MountingHole_3.2mm_M3, Mounting_Holes:MountingHole_3.2mm_M3, F.Cu at (95.4, 62.0)
- moved JP4 0.38 mm to (97.2, 68.8)
- moved JP4 0.32 mm to (147.1, 67.3)
Connections:
- JP4 pad 1: GNDPWR -> GNDS
Routing:
- net GNDS: track 432.0 -> 449.4 mm, vias 78 -> 88
- net (no net): track 0.00 -> 7.19 mm, vias 0 -> 3
Other:
- outline, holes or cut-outs redrawn
