File: Arm_stepper.kicad_pcb (KiCad board)
At the start: 2 copper layers, 178.3 x 60.5 mm, 129 parts, among them IC1 L6208D, J1 12V_CONN, J10 ENCODER1, J11 ENCODER2, J3 M1_CONN, J4 Conn_01x06_Male, J5 I2C_CONN, J8 Conn_01x04_Female, J9 USB_B_Mini, M2 Fan, Q2 2N2219, SW1 SW_Push_Dual, SW2 endstop4, SW3 endstop1, SW4 endstop3, SW5 endstop2, U1 ISO1050-00_isolation, U2 USBLC6-2SC6, U3 STM32F446RETx, U4 LM1117-3.3, U5 LM1117-5, Y1 8Mhz

Commit message: little fix
Routing:
- net GNDS: track 449.4 -> 457.9 mm, vias 88 -> 91
- net (no net): track 7.19 -> 0.27 mm, vias 3 -> 0
Changed lines of the file:
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@@
     (thickness 1.6)
     (drawings 30)
-    (tracks 2497)
+    (tracks 2498)
     (zones 0)
     (modules 129)
@@
   (layers
     (0 F.Cu signal)
-    (31 B.Cu signal)
+    (31 B.Cu signal hide)
     (32 B.Adhes user)
     (33 F.Adhes user)
@@
   )
   (setup
-    (last_trace_width 2.5)
+    (last_trace_width 0.9)
     (user_trace_width 0.25)
     (user_trace_width 0.4)
@@
   (gr_poly (pts (xy 139.5095 81.5975) (xy 145.8595 81.4705) (xy 145.796 69.1896) (xy 125.222 69.0372) (xy 125.4252 81.026) (xy 128.1176 81.1784) (xy 135.8265 81.4705)) (layer F.Mask) (width 0.15))
   (gr_poly (pts (xy 133.477 99.187) (xy 125.6665 99.7585) (xy 125.6665 107.2515) (xy 151.5745 107.2515) (xy 151.5364 99.4664)) (layer F.Mask) (width 0.15))
-  (via (at 162.2425 106.299) (size 0.8) (drill 0.4) (layers F.Cu B.Cu) (net 0))
-  (segment (start 162.306 106.2355) (end 162.2425 106.299) (width 0.25) (layer B.Cu) (net 0))
-  (segment (start 162.2425 106.299) (end 163.322 107.3785) (width 0.7) (layer F.Cu) (net 0))
-  (via (at 165.862 108.5215) (size 0.8) (drill 0.4) (layers F.Cu B.Cu) (net 0))
-  (segment (start 164.719 107.3785) (end 165.862 108.5215) (width 0.7) (layer F.Cu) (net 0))
-  (segment (start 163.322 107.3785) (end 164.719 107.3785) (width 0.7) (layer F.Cu) (net 0))
-  (via (at 166.0525 106.1085) (size 0.8) (drill 0.4) (layers F.Cu B.Cu) (net 0))
-  (segment (start 165.989 106.1085) (end 166.0525 106.1085) (width 0.25) (layer B.Cu) (net 0))
-  (segment (start 166.0525 108.331) (end 165.862 108.5215) (width 0.25) (layer F.Cu) (net 0))
-  (segment (start 166.0525 106.1085) (end 166.0525 108.331) (width 0.7) (layer F.Cu) (net 0))
+  (via (at 162.1155 106.045) (size 0.8) (drill 0.4) (layers F.Cu B.Cu) (net 1))
+  (segment (start 162.306 106.2355) (end 162.1155 106.045) (width 0.9) (layer B.Cu) (net 0))
   (segment (start 136.8285 67.1195) (end 137.0965 67.1195) (width 3) (layer F.Cu) (net 1))
   (segment (start 122.4225 67.1195) (end 133.4135 67.1195) (width 3) (layer F.Cu) (net 1))
@@
   (segment (start 165.92301 71.882) (end 165.989 71.81601) (width 1.1) (layer F.Cu) (net 1))
   (segment (start 161.9885 71.882) (end 165.92301 71.882) (width 1.1) (layer F.Cu) (net 1))
+  (via (at 166.243 105.9815) (size 0.8) (drill 0.4) (layers F.Cu B.Cu) (net 1))
+  (segment (start 166.243 106.054318) (end 166.243 105.9815) (width 0.9) (layer F.Cu) (net 1))
+  (segment (start 162.909825 107.40501) (end 164.892308 107.40501) (width 0.9) (layer F.Cu) (net 1))
+  (segment (start 162.1155 106.610685) (end 162.909825 107.40501) (width 0.9) (layer F.Cu) (net 1))
+  (segment (start 164.892308 107.40501) (end 166.243 106.054318) (width 0.9) (layer F.Cu) (net 1))
+  (segment (start 162.1155 106.045) (end 162.1155 106.610685) (width 0.9) (layer F.Cu) (net 1))
+  (segment (start 166.243 108.7755) (end 166.1795 108.839) (width 0.9) (layer F.Cu) (net 1))
+  (via (at 166.1795 108.839) (size 0.8) (drill 0.4) (layers F.Cu B.Cu) (net 1))
+  (segment (start 166.243 105.9815) (end 166.243 108.7755) (width 0.9) (layer F.Cu) (net 1))
   (segment (start 74.9295 68.9365) (end 75.1205 68.7455) (width 1.1) (layer F.Cu) (net 2))
   (segment (start 74.9295 71.6915) (end 74.9295 68.9365) (width 1.1) (layer F.Cu) (net 2))

Commit message: improve
Routing:
- net GNDD: track 0.00 -> 407.3 mm
- net GNDS: track 457.9 -> 421.8 mm, vias 91 -> 100
- net t_SENS: track 51.4 -> 49.2 mm
- net CLK1: track 194.5 -> 193.7 mm
- added copper zone on F.Cu, net GNDS
Other:
- outline, holes or cut-outs redrawn

Commit message: init
Parts:
- removed the C13 at (170.9, 88.0)
- removed the C13 at (103.2, 88.1)
- removed the C17 at (170.9, 99.4)
- removed the C17 at (103.2, 99.5)
- removed the C21 at (203.0, 65.0)
- removed the C21 at (135.3, 65.1)
- removed the C22 at (206.8, 65.1)
- removed the C22 at (139.1, 65.1)
- removed the C23 at (221.0, 83.7)
- removed the C23 at (153.4, 83.7)
- removed the C24 at (188.0, 83.7)
- removed the C24 at (120.3, 83.7)
- removed the C28 at (225.9, 101.9)
- removed the C28 at (158.2, 101.9)
- removed the C3 at (186.1, 95.8)
- removed the C3 at (118.4, 95.8)
- removed the C30 at (186.1, 102.0)
- removed the C30 at (118.4, 102.0)
- removed the C7 at (223.8, 97.2)
- removed the C7 at (156.1, 97.2)
- removed the D1 at (167.7, 92.5)
- removed the D1 at (100.0, 92.5)
- removed the D15 at (216.2, 112.3)
- removed the D15 at (148.5, 112.3)
- removed the D16 at (185.0, 115.1)
- removed the D16 at (117.3, 115.1)
- removed the D17 at (223.8, 115.6)
- removed the D17 at (156.1, 115.6)
- removed the D18 at (177.9, 115.1)
- removed the D18 at (110.2, 115.1)
- removed the D5 at (174.1, 92.5)
- removed the D5 at (106.4, 92.5)
- removed HS1 (x4): Heatsink_Pad, SMD_Packages:1Pin
- removed the IC1 at (204.5, 89.9)
- removed the IC1 at (136.8, 90.0)
- removed the J3 at (199.5, 114.0)
- removed the J3 at (131.8, 114.1)
- removed the JP4 at (147.1, 67.3)
- removed the JP4 at (97.2, 68.8)
- removed the M2 at (177.4, 70.9)
- removed the M2 at (113.1, 70.0)
- removed the R10 at (177.9, 97.5)
- removed the R10 at (110.2, 97.6)
- removed the R12 at (217.9, 83.6)
- removed the R12 at (150.2, 83.6)
- removed the R13 at (184.8, 83.6)
- removed the R13 at (117.2, 83.6)
- removed the R14 at (226.1, 84.6)
- removed the R14 at (158.4, 84.6)
- removed the R17 at (179.8, 84.2)
- removed the R17 at (112.1, 84.3)
- removed the R19 at (225.9, 105.2)
- removed the R19 at (158.2, 105.2)
- removed the R25 at (186.0, 105.2)
- removed the R25 at (118.3, 105.2)
- removed the R34 at (223.8, 110.2)
- removed the R34 at (156.1, 110.3)
- removed the R35 at (188.0, 110.2)
- removed the R35 at (120.3, 110.3)
- removed the R4 at (186.0, 98.8)
- removed the R4 at (118.3, 98.9)
- removed the R41 at (216.2, 114.8)
- removed the R41 at (148.5, 114.9)
- removed the R42 at (185.0, 117.9)
- removed the R42 at (117.3, 117.9)
- removed the R43 at (216.2, 117.6)
- removed the R43 at (148.5, 117.7)
- removed the R44 at (177.9, 117.9)
- removed the R44 at (110.2, 117.9)
- removed REF** (x4): MountingHole_3.2mm_M3, Mounting_Holes:MountingHole_3.2mm_M3
- added C13: 220nF1, Capacitor_SMD:C_0805_2012Metric, F.Cu at (138.0, 114.5)
- added C15: 220nF1, Capacitor_SMD:C_0805_2012Metric, F.Cu at (240.9, 51.7)
- added C17: 10nF, Capacitor_SMD:C_0805_2012Metric, F.Cu at (138.0, 120.5)
- added C18: 5.6n, Capacitor_SMD:C_0805_2012Metric, F.Cu at (261.0, 39.4)
- added C19: 100nF, Capacitor_SMD:C_0805_2012Metric, F.Cu at (246.0, 48.6)
- added C20: 10nF, Capacitor_SMD:C_0805_2012Metric, F.Cu at (240.9, 53.6)
- added C21: 100nF, Capacitor_SMD:C_1210_3225Metric, F.Cu at (114.6, 106.6)
- added C22: 100uF ceramic, Capacitor_SMD:C_1210_3225Metric, F.Cu at (118.1, 106.6)
- added C23: 1nF, Capacitor_SMD:C_0805_2012Metric, F.Cu at (105.0, 133.0)
- added C24: 1nF, Capacitor_SMD:C_0805_2012Metric, F.Cu at (128.0, 133.0)
- added C25: 100nF, Capacitor_SMD:C_1206_3216Metric_Pad1.42x1.75mm_HandSolder, F.Cu at (236.7, 51.8)
- added C28: 68nF, Capacitor_SMD:C_0805_2012Metric, F.Cu at (98.0, 128.0)
- added C29: 100uF ceramic, Capacitor_SMD:C_1206_3216Metric_Pad1.42x1.75mm_HandSolder, F.Cu at (276.9, 10.9)
- added C3: 5.6n, Capacitor_SMD:C_0805_2012Metric, F.Cu at (135.0, 126.0)
- added C30: 68nF, Capacitor_SMD:C_0805_2012Metric, F.Cu at (139.0, 126.0)
- added C32: 1nF, Capacitor_SMD:C_0805_2012Metric, F.Cu at (247.7, 54.4)
- added C33: 1nF, Capacitor_SMD:C_0805_2012Metric, F.Cu at (276.3, 25.8)
- added C36: 68nF, Capacitor_SMD:C_0805_2012Metric, F.Cu at (249.4, 46.6)
- added C38: 68nF, Capacitor_SMD:C_0805_2012Metric, F.Cu at (254.1, 40.7)
- added C7: 100nF, Capacitor_SMD:C_0805_2012Metric, F.Cu at (98.0, 125.0)
- added D1: 1N4148, Diode_SMD:D_SOD-123, F.Cu at (135.0, 117.5)
- added D10: LED_RED, LED_SMD:LED_0805_2012Metric, F.Cu at (275.1, 15.1)
- added D11: LED, LED_SMD:LED_0805_2012Metric, F.Cu at (275.1, 17.1)
- added D12: LED, LED_SMD:LED_0805_2012Metric, F.Cu at (258.8, 33.5)
- added D13: LED, LED_SMD:LED_0805_2012Metric, F.Cu at (270.4, 21.9)
- added D14: LED, LED_SMD:LED_0805_2012Metric, F.Cu at (252.9, 38.7)
- added D15: LED, LED_SMD:LED_0805_2012Metric, F.Cu at (104.0, 150.0)
- added D16: LED, LED_SMD:LED_0805_2012Metric, F.Cu at (129.0, 150.0)
- added D17: LED, LED_SMD:LED_0805_2012Metric, F.Cu at (103.9, 144.0)
- added D18: LED, LED_SMD:LED_0805_2012Metric, F.Cu at (129.1, 144.0)
- added D4: 1N4148, Diode_SMD:D_SOD-123, F.Cu at (246.7, 42.1)
- added D5: 1N4148, Diode_SMD:D_SOD-123, F.Cu at (141.0, 117.5)
- added D6: 1N4148, Diode_SMD:D_SOD-123, F.Cu at (236.6, 54.1)
- added D8: 1N4148, Diode_SMD:D_SOD-123, F.Cu at (241.6, 49.5)
- added IC1: L6208D, T0-R0_Stepper_Board:POWERSO36, F.Cu at (116.0, 127.0)
- added IC2: L6208D, T0-R0_Stepper_Board:POWERSO36, F.Cu at (233.7, 17.5)
- added J2: M1_CONN, TerminalBlock_Phoenix:TerminalBlock_Phoenix_PT-1,5-4-3.5-H_1x04_P3.50mm_Horizontal, F.Cu at (226.0, 28.8)
- added J3: M1_CONN, TerminalBlock_Phoenix:TerminalBlock_Phoenix_PT-1,5-4-3.5-H_1x04_P3.50mm_Horizontal, F.Cu at (111.0, 151.0)
- added JP1: Jumper_NO_Small, Connector_PinSocket_2.54mm:PinSocket_1x02_P2.54mm_Vertical, F.Cu at (261.1, 24.8)
- added JP4: SolderJumper_2_Bridged, Connector_Wire:SolderWirePad_1x02_P5.08mm_Drill1.5mm, F.Cu at (131.0, 99.0)
- added JP5: SolderJumper_2_Bridged, Connector_Wire:SolderWirePad_1x02_P5.08mm_Drill1.5mm, F.Cu at (259.4, 12.0)
- added L1: L, Inductor_SMD:L_1206_3216Metric_Pad1.42x1.75mm_HandSolder, F.Cu at (236.7, 49.5)
- added M2: Fan, Connector_PinSocket_2.54mm:PinSocket_1x02_P2.54mm_Vertical, F.Cu at (248.3, 34.3)
- added R10: 100, Resistor_SMD:R_0805_2012Metric, F.Cu at (138.0, 123.5)
- added R11: 100, Resistor_SMD:R_0805_2012Metric, F.Cu at (257.6, 40.6)
- added R12: 39k, Resistor_SMD:R_0805_2012Metric, F.Cu at (102.0, 133.0)
- added R13: 39k, Resistor_SMD:R_0805_2012Metric, F.Cu at (131.0, 133.0)
- added R14: 0.3, Resistor_SMD:R_2512_6332Metric, F.Cu at (103.0, 125.7)
- added R15: 39k, Resistor_SMD:R_0805_2012Metric, F.Cu at (243.3, 55.6)
- added R16: 39k, Resistor_SMD:R_0805_2012Metric, F.Cu at (271.4, 27.8)
- added R17: 0.3, Resistor_SMD:R_2512_6332Metric, F.Cu at (130.0, 126.0)
- added R18: 0.3, Resistor_SMD:R_2512_6332Metric, F.Cu at (270.6, 11.7)
- added R19: 2.2K, Resistor_SMD:R_0805_2012Metric, F.Cu at (98.0, 131.0)
- added R20: 0.3, Resistor_SMD:R_2512_6332Metric, F.Cu at (242.6, 38.3)
- added R22: 1k, Resistor_SMD:R_0805_2012Metric, F.Cu at (252.8, 46.6)
- added R23: 4.7K, Resistor_SMD:R_0805_2012Metric, F.Cu at (276.3, 23.8)
- added R25: 2.2K, Resistor_SMD:R_0805_2012Metric, F.Cu at (139.1, 129.0)
- added R26: 2.2K, Resistor_SMD:R_0805_2012Metric, F.Cu at (252.8, 48.5)
- added R33: 2.2K, Resistor_SMD:R_0805_2012Metric, F.Cu at (269.0, 33.7)
- added R34: 4.7K, Resistor_SMD:R_0805_2012Metric, F.Cu at (98.0, 133.2)
- added R35: 4.7K, Resistor_SMD:R_0805_2012Metric, F.Cu at (269.0, 31.7)
- added R36: 4.7K, Resistor_SMD:R_0805_2012Metric, F.Cu at (256.2, 48.5)
- added R37: 10K, Resistor_SMD:R_0805_2012Metric, F.Cu at (269.0, 35.6)
- added R38: 10K, Resistor_SMD:R_0805_2012Metric, F.Cu at (261.0, 43.3)
- added R39: 10K, Resistor_SMD:R_0805_2012Metric, F.Cu at (264.4, 39.4)
- added R4: 100k, Resistor_SMD:R_0805_2012Metric, F.Cu at (135.0, 129.0)
- added R40: 10K, Resistor_SMD:R_0805_2012Metric, F.Cu at (246.7, 56.4)
- added R41: 10K, Resistor_SMD:R_0805_2012Metric, F.Cu at (104.0, 147.0)
- added R42: 10K, Resistor_SMD:R_0805_2012Metric, F.Cu at (128.9, 147.0)
- added R43: 10K, Resistor_SMD:R_0805_2012Metric, F.Cu at (104.0, 141.0)
- added R44: 10K, Resistor_SMD:R_0805_2012Metric, F.Cu at (129.0, 141.0)
- added R9: 100k, Resistor_SMD:R_0805_2012Metric, F.Cu at (254.1, 44.6)
- C1, C10, C11, C12, C14, C2, C26, C27, C34, C35, C4, C5, C8, C9: footprint Capacitors_SMD:C_1206_HandSoldering -> Capacitor_SMD:C_0805_2012Metric
- D2: footprint LEDs:LED_RGB_1210 -> LED_SMD:LED_RGB_1210
- D9: footprint LEDs:LED_1206_HandSoldering -> LED_SMD:LED_0805_2012Metric
- J1: footprint TerminalBlocks_Phoenix:TerminalBlock_Phoenix_PT-3.5mm_2pol -> TerminalBlock_Phoenix:TerminalBlock_Phoenix_PT-1,5-2-3.5-H_1x02_P3.50mm_Horizontal
- J10, J11: footprint TerminalBlocks_Phoenix:TerminalBlock_Phoenix_MPT-2.54mm_4pol -> TerminalBlock_Phoenix:TerminalBlock_Phoenix_MPT-0,5-4-2.54_1x04_P2.54mm_Horizontal
- J4: footprint Pin_Headers:Pin_Header_Angled_1x06_Pitch2.54mm -> Connector_PinHeader_2.54mm:PinHeader_1x06_P2.54mm_Vertical
- J5: footprint TerminalBlocks_Phoenix:TerminalBlock_Phoenix_MPT-2.54mm_2pol -> TerminalBlock_Phoenix:TerminalBlock_Phoenix_MPT-0,5-4-2.54_1x04_P2.54mm_Horizontal
- J8: footprint TerminalBlocks_Phoenix:TerminalBlock_Phoenix_MPT-2.54mm_4pol -> Connector_Dsub:DSUB-9_Female_Horizontal_P2.77x2.84mm_EdgePinOffset4.94mm_Housed_MountingHolesOffset7.48mm
- J9: footprint Connectors_USB:USB_Micro-B_Molex-105017-0001 -> Connector_USB:USB_Micro-B_Molex-105017-0001
- Q2: footprint TO_SOT_Packages_SMD:SOT-23 -> Package_TO_SOT_SMD:SOT-23_Handsoldering
- R1, R2, R21, R24, R28, R29, R3, R30, R31, R32, R45, R46, R47, R48, R5, R6, R7, TH1: footprint Resistors_SMD:R_1206_HandSoldering -> Resistor_SMD:R_0805_2012Metric
- SW1: footprint Buttons_Switches_THT:SW_TH_Tactile_Omron_B3F-10xx -> Button_Switch_SMD:SW_SPST_B3S-1000
- SW2, SW3, SW4, SW5: footprint TerminalBlocks_Phoenix:TerminalBlock_Phoenix_MPT-2.54mm_2pol -> TerminalBlock_Phoenix:TerminalBlock_Phoenix_MPT-0,5-2-2.54_1x02_P2.54mm_Horizontal
- U1: footprint ISO1050:SO8 -> Package_SO:SSO-8_6.7x9.8mm_P2.54mm_Clearance8mm
- U2: footprint TO_SOT_Packages_SMD:SOT-23-6_Handsoldering -> Package_TO_SOT_SMD:SOT-23-6_Handsoldering
- U3: footprint Housings_QFP:LQFP-64_10x10mm_Pitch0.5mm -> Package_QFP:LQFP-64_10x10mm_P0.5mm
- U4, U5: footprint TO_SOT_Packages_SMD:SOT-223-3_TabPin2 -> Package_TO_SOT_SMD:SOT-223-3_TabPin2
- Y1: footprint Crystals:Crystal_HC49-U_Vertical -> Crystal:Crystal_HC49-4H_Vertical
- moved C9 226.3 mm to (278.5, 15.1), turned to 0 degrees
- moved C10 225.1 mm to (275.1, 19.1), turned to 0 degrees
- moved C8 220.5 mm to (278.5, 17.0), turned to 0 degrees
- moved R47 218.0 mm to (278.3, 27.7), turned to 0 degrees
- moved U2 210.6 mm to (265.3, 24.8), turned to 0 degrees
- moved SW2 208.5 mm to (268.8, 17.3)
- moved J1 206.3 mm to (259.4, 17.9), turned to 0 degrees
- moved R6 201.9 mm to (278.5, 19.0)
- moved R3 201.7 mm to (262.2, 35.5), turned to 0 degrees
- moved C11 197.0 mm to (258.7, 35.5)
- moved R30 195.4 mm to (277.2, 21.1), turned to 0 degrees
- moved D9 195.0 mm to (258.8, 31.5), turned to 0 degrees
- moved R48 194.3 mm to (259.8, 37.5), turned to 0 degrees
- moved J11 194.0 mm to (240.8, 28.8)
- moved C1 192.4 mm to (262.2, 33.5), turned to 0 degrees
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Connections:
- R1 pad 1: Net-(J8-Pad2) -> Net-(JP1-Pad2)
Routing:
- net GNDS: track 421.8 -> 0.00 mm, vias 100 -> 0
- net GNDD: track 407.3 -> 0.00 mm, vias 776 -> 0
- net +12V: track 429.1 -> 76.7 mm, vias 1 -> 0
- net +3V3: track 242.3 -> 0.00 mm, vias 35 -> 0
- net CW1: track 216.3 -> 0.00 mm, vias 5 -> 0
- net CLK1: track 193.7 -> 0.00 mm, vias 5 -> 0
- net CRTL1: track 228.1 -> 42.1 mm, vias 3 -> 2
- net PWMA1: track 182.2 -> 17.7 mm, vias 4 -> 0
- net Net-(C3-Pad1): track 174.7 -> 15.1 mm, vias 6 -> 0
- net /NRST: track 157.7 -> 0.00 mm, vias 3 -> 0
- net RST1: track 167.1 -> 10.6 mm, vias 6 -> 0
- net HALF1: track 186.3 -> 39.6 mm, vias 7 -> 2
- net +5V: track 127.7 -> 0.00 mm, vias 18 -> 0
- net PWMB1: track 126.9 -> 0.00 mm, vias 4 -> 0
- net Net-(C30-Pad2): track 123.3 -> 24.6 mm, vias 6 -> 0
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- removed copper zone on B.Cu, net +3V3
- removed copper zone on F.Cu, net +3V3
- removed copper zone on B.Cu, net GNDD
- removed copper zone on F.Cu, net GNDD
- removed copper zone on B.Cu, net GNDS
- removed copper zone on F.Cu, net GNDS
Other:
- board outline removed
- rule pad_to_mask_clearance: 0.051 -> 0
- board text added: "A+ A- B- B+"

Commit message: work
Parts:
- JP4: footprint Connector_Wire:SolderWirePad_1x02_P5.08mm_Drill1.5mm -> Wire_Connections_Bridges:WireConnection_1.50mmDrill
- moved C9 245.6 mm to (57.9, 122.9), turned to 90 degrees
- moved C10 243.9 mm to (57.9, 130.2), turned to 90 degrees
- moved C8 231.5 mm to (70.1, 117.6), turned to 180 degrees
- moved D9 230.2 mm to (46.4, 120.1), turned to 90 degrees
- moved U2 230.1 mm to (41.1, 76.7), turned to 270 degrees
- moved R47 222.5 mm to (73.6, 115.1), turned to 180 degrees
- moved C11 217.5 mm to (43.4, 66.3), turned to 270 degrees
- moved R45 216.8 mm to (39.4, 72.1)
- moved R3 215.6 mm to (67.9, 129.0), turned to 180 degrees
- moved JP1 213.9 mm to (48.5, 48.8), turned to 270 degrees
- moved C12 212.5 mm to (80.9, 136.6), turned to 270 degrees
- moved R6 212.5 mm to (91.4, 119.6)
- moved R21 211.9 mm to (46.4, 116.5), turned to 90 degrees
- moved C34 211.6 mm to (50.0, 116.5), turned to 270 degrees
- moved J9 209.7 mm to (26.2, 76.7), turned to 270 degrees
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- renumbered M2 to FAN
Routing:
- net GNDD: track 0.00 -> 223.3 mm, vias 0 -> 156
- net +12V: track 76.7 -> 192.0 mm
- net /NRST: track 0.00 -> 73.5 mm
- net GNDS: track 0.00 -> 71.3 mm, vias 0 -> 67
- net PWMB1: track 0.00 -> 64.2 mm, vias 0 -> 2
- net GNDPWR: track 0.00 -> 62.8 mm, vias 0 -> 2
- net t_SENS: track 0.00 -> 59.8 mm, vias 0 -> 2
- net Net-(R5-Pad2): track 0.00 -> 30.1 mm
- net /TRACESWO: track 0.00 -> 28.5 mm
- net Net-(R6-Pad2): track 0.00 -> 21.9 mm
- net Net-(C8-Pad2): track 0.00 -> 17.8 mm
- net /SWCLK: track 0.00 -> 17.6 mm
- net /SWDIO: track 0.00 -> 15.8 mm
- net Net-(R7-Pad2): track 0.00 -> 15.2 mm
- net Net-(C9-Pad1): track 0.00 -> 14.5 mm
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- added copper zone on F.Cu, net GNDD
- added copper zone on B.Cu, net GNDS
- added copper zone on F.Cu, net GNDS
Other:
- board text added: "+"
- board text added: "-"

Commit message: 2.
Parts:
- added C13: 220nF1, Capacitor_SMD:C_0805_2012Metric, F.Cu at (395.8, 112.0)
- added C17: 10nF, Capacitor_SMD:C_0805_2012Metric, F.Cu at (395.8, 118.0)
- added C21: 100nF, Capacitor_SMD:C_1210_3225Metric, F.Cu at (372.4, 104.0)
- added C22: 100uF ceramic, Capacitor_SMD:C_1210_3225Metric, F.Cu at (375.9, 104.0)
- added C23: 1nF, Capacitor_SMD:C_0805_2012Metric, F.Cu at (362.8, 130.5)
- added C24: 1nF, Capacitor_SMD:C_0805_2012Metric, F.Cu at (385.8, 130.5)
- added C28: 68nF, Capacitor_SMD:C_0805_2012Metric, F.Cu at (355.9, 126.5)
- added C3: 5.6n, Capacitor_SMD:C_0805_2012Metric, F.Cu at (392.8, 123.5)
- added C30: 68nF, Capacitor_SMD:C_0805_2012Metric, F.Cu at (396.8, 123.5)
- added C7: 100nF, Capacitor_SMD:C_0805_2012Metric, F.Cu at (354.8, 124.5)
- added D1: 1N4148, Diode_SMD:D_SOD-123, F.Cu at (392.8, 115.0)
- added D15: LED, LED_SMD:LED_0805_2012Metric, F.Cu at (361.8, 147.5)
- added D16: LED, LED_SMD:LED_0805_2012Metric, F.Cu at (386.8, 147.5)
- added D17: LED, LED_SMD:LED_0805_2012Metric, F.Cu at (361.7, 141.5)
- added D18: LED, LED_SMD:LED_0805_2012Metric, F.Cu at (386.9, 141.5)
- added D5: 1N4148, Diode_SMD:D_SOD-123, F.Cu at (398.8, 115.0)
- added IC1: L6208D, T0-R0_Stepper_Board:POWERSO36, F.Cu at (373.8, 124.5)
- added J3: M1_CONN, TerminalBlock_Phoenix:TerminalBlock_Phoenix_PT-1,5-4-3.5-H_1x04_P3.50mm_Horizontal, F.Cu at (368.8, 148.5)
- added JP4: SolderJumper_2_Bridged, Wire_Connections_Bridges:WireConnection_1.50mmDrill, F.Cu at (380.5, 92.5)
- added R10: 100, Resistor_SMD:R_0805_2012Metric, F.Cu at (395.8, 121.0)
- added R12: 39k, Resistor_SMD:R_0805_2012Metric, F.Cu at (359.8, 130.5)
- added R13: 39k, Resistor_SMD:R_0805_2012Metric, F.Cu at (388.8, 130.5)
- added R14: 0.3, Resistor_SMD:R_2512_6332Metric, F.Cu at (360.8, 123.2)
- added R17: 0.3, Resistor_SMD:R_2512_6332Metric, F.Cu at (387.8, 123.5)
- added R19: 2.2K, Resistor_SMD:R_0805_2012Metric, F.Cu at (355.8, 128.5)
- added R24: 27K, Resistor_SMD:R_0805_2012Metric, F.Cu at (385.0, 112.2)
- added R25: 2.2K, Resistor_SMD:R_0805_2012Metric, F.Cu at (396.9, 126.5)
- added R34: 4.7K, Resistor_SMD:R_0805_2012Metric, F.Cu at (355.8, 130.7)
- added R35: 4.7K, Resistor_SMD:R_0805_2012Metric, F.Cu at (395.6, 128.8)
- added R4: 100k, Resistor_SMD:R_0805_2012Metric, F.Cu at (392.8, 126.5)
- added R41: 10K, Resistor_SMD:R_0805_2012Metric, F.Cu at (361.8, 144.5)
- added R42: 10K, Resistor_SMD:R_0805_2012Metric, F.Cu at (386.7, 144.5)
- added R43: 10K, Resistor_SMD:R_0805_2012Metric, F.Cu at (361.8, 138.5)
- added R44: 10K, Resistor_SMD:R_0805_2012Metric, F.Cu at (386.8, 138.5)
- added SW2: endstop4, TerminalBlock_Phoenix:TerminalBlock_Phoenix_MPT-0,5-2-2.54_1x02_P2.54mm_Horizontal, F.Cu at (353.1, 149.9)
- added TH1: 10k+30T, Resistor_SMD:R_0805_2012Metric, F.Cu at (385.0, 115.8)
- J5: footprint TerminalBlock_Phoenix:TerminalBlock_Phoenix_MPT-0,5-4-2.54_1x04_P2.54mm_Horizontal -> TerminalBlocks_Phoenix:TerminalBlock_Phoenix_MPT-2.54mm_2pol
- moved R30 231.3 mm to (82.5, 146.1), turned to 270 degrees
- moved C1 220.1 mm to (54.6, 106.7), turned to 270 degrees
- moved SW2 220.0 mm to (95.2, 152.4)
- moved C4 216.0 mm to (59.7, 106.7), turned to 270 degrees
- moved J11 215.0 mm to (64.8, 152.4)
- moved R32 212.4 mm to (76.2, 146.1), turned to 270 degrees
- moved R29 209.1 mm to (95.2, 146.1), turned to 270 degrees
- moved R28 208.4 mm to (88.9, 146.1), turned to 270 degrees
- moved C27 207.7 mm to (83.8, 142.2), turned to 180 degrees
- moved SW3 207.0 mm to (82.5, 152.4)
- moved C5 205.7 mm to (62.2, 106.7), turned to 270 degrees
- moved J10 200.3 mm to (53.3, 152.4)
- moved U5 199.7 mm to (90.2, 139.7)
- moved C14 199.0 mm to (68.3, 121.3), turned to 180 degrees
- moved SW5 195.8 mm to (76.2, 152.4)
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Connections:
- J10 pad 1: E1_2 -> +5V
- J10 pad 2: +5V -> E1_2
- J11 pad 1: E2_2 -> +5V
- J11 pad 2: +5V -> E2_2
Routing:
- net +12V: track 192.0 -> 555.6 mm
- net GNDD: track 223.3 -> 446.6 mm, vias 156 -> 312
- net +3V3: track 3.13 -> 114.4 mm, vias 0 -> 12
- net GNDS: track 71.3 -> 157.7 mm, vias 67 -> 155
- net +5V: track 0.00 -> 66.8 mm, vias 0 -> 5
- net USB_DP: track 0.00 -> 65.9 mm
- net i2C1_SCL: track 0.00 -> 60.1 mm, vias 0 -> 2
- net GNDPWR: track 62.8 -> 122.6 mm
- net CW1: track 0.00 -> 57.5 mm, vias 0 -> 4
- net CLK1: track 0.00 -> 56.3 mm, vias 0 -> 4
- net PWMB1: track 64.2 -> 115.7 mm, vias 2 -> 3
- net FAN: track 0.00 -> 49.2 mm, vias 0 -> 2
- net E1_1: track 0.00 -> 45.7 mm
- net E4: track 0.00 -> 45.1 mm
- net /M2_A-: track 43.8 -> 87.6 mm, vias 2 -> 4
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
Commit message: 2.2
Routing:
- net i2C1_SDA: track 5.66 -> 56.4 mm
Changed lines of the file:
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@@
     (thickness 1.6)
     (drawings 12)
-    (tracks 1667)
+    (tracks 1678)
     (zones 0)
     (modules 161)
@@
   (segment (start 78.85 113.6988) (end 78.85 121.525) (width 0.25) (layer F.Cu) (net 64))
   (segment (start 77.476601 112.325401) (end 78.85 113.6988) (width 0.25) (layer F.Cu) (net 64))
-  (via (at 74.3 116.925) (size 0.8) (drill 0.4) (layers F.Cu B.Cu) (net 65))
   (segment (start 74.3 117.686002) (end 74.3 116.925) (width 0.2) (layer F.Cu) (net 65))
   (segment (start 76.85 120.236002) (end 74.3 117.686002) (width 0.2) (layer F.Cu) (net 65))
   (segment (start 76.85 121.525) (end 76.85 120.236002) (width 0.2) (layer F.Cu) (net 65))
+  (segment (start 77.604001 115.295999) (end 75.975 116.925) (width 0.2) (layer B.Cu) (net 65))
+  (segment (start 77.604001 110.598399) (end 77.604001 115.295999) (width 0.2) (layer B.Cu) (net 65))
+  (segment (start 77.006001 110.000399) (end 77.604001 110.598399) (width 0.2) (layer B.Cu) (net 65))
+  (segment (start 75.0317 110.000399) (end 77.006001 110.000399) (width 0.2) (layer B.Cu) (net 65))
+  (segment (start 70.0813 105.049999) (end 75.0317 110.000399) (width 0.2) (layer B.Cu) (net 65))
+  (segment (start 41.83949 111.76) (end 42.689491 110.909999) (width 0.2) (layer B.Cu) (net 65))
+  (segment (start 42.689491 110.909999) (end 54.853999 110.909999) (width 0.2) (layer B.Cu) (net 65))
+  (segment (start 60.713999 105.049999) (end 70.0813 105.049999) (width 0.2) (layer B.Cu) (net 65))
+  (via (at 75.975 116.925) (size 0.8) (drill 0.4) (layers F.Cu B.Cu) (net 65))
+  (segment (start 54.853999 110.909999) (end 60.713999 105.049999) (width 0.2) (layer B.Cu) (net 65))
+  (segment (start 40.64 111.76) (end 41.83949 111.76) (width 0.2) (layer B.Cu) (net 65))
+  (segment (start 75.975 116.925) (end 74.3 116.925) (width 0.2) (layer F.Cu) (net 65))
   (via (at 56.45 111.775) (size 0.8) (drill 0.4) (layers F.Cu B.Cu) (net 66))
   (segment (start 49.356516 118.18401) (end 53.132484 118.18401) (width 0.2) (layer F.Cu) (net 66))

Commit message: dual
Parts:
- moved C12 0.53 mm to (80.4, 136.6)
Connections:
- J8 pad 1: /+5v_can -> (no net)
- J8 pad 2: Net-(J8-Pad2) -> Net-(J8-Pad3)
- J8 pad 3: Net-(J8-Pad3) -> /gnd_can
- J8 pad 4: /gnd_can -> (no net)
- J8 pad 7: (no net) -> Net-(J8-Pad2)
- J8 pad 9: (no net) -> /+5v_can
Routing:
- net GNDS: track 157.7 -> 176.0 mm, vias 155 -> 214
- net Net-(JP1-Pad2): track 22.0 -> 6.76 mm, vias 0 -> 1
- net /+5v_can: track 14.1 -> 24.4 mm
- net Net-(J8-Pad2): track 26.1 -> 28.4 mm
- net CLK1: track 56.3 -> 58.4 mm
- net /gnd_can: track 13.4 -> 14.5 mm
- net E2_2: track 37.5 -> 38.2 mm
- net E1_2: vias 2 -> 3

Commit message: duala
Parts:
- removed the SW2 at (353.1, 149.9)
- moved C7 209.0 mm to (145.8, 127.0)
- moved JP4 209.0 mm to (171.5, 95.0)
- moved C13 209.0 mm to (186.8, 114.5)
- moved C17 209.0 mm to (186.8, 120.5)
- moved C23 209.0 mm to (153.8, 133.0)
- moved C24 209.0 mm to (176.8, 133.0)
- moved C3 209.0 mm to (183.8, 126.0)
- moved C30 209.0 mm to (187.8, 126.0)
- moved D1 209.0 mm to (183.8, 117.5)
- moved D15 209.0 mm to (152.8, 150.0)
- moved D16 209.0 mm to (177.8, 150.0)
- moved D17 209.0 mm to (152.7, 144.0)
- moved D18 209.0 mm to (177.9, 144.0)
- moved D5 209.0 mm to (189.8, 117.5)
- moved IC1 209.0 mm to (164.8, 127.0)
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Routing:
- net +12V: track 555.6 -> 521.7 mm
- net GNDPWR: track 122.6 -> 138.0 mm
Other:
- board outline added: 154.5 x 60 mm
