File: Arm_stepper.kicad_pcb (KiCad board)
At the start: 2 copper layers, 154.5 x 60 mm, 160 parts, among them IC1 L6208D, IC2 L6208D, J1 12V_CONN, J10 ENCODER1, J11 ENCODER2, J2 M1_CONN, J3 M1_CONN, J4 Conn_01x06_Male, J5 I2C_CONN, J8 Conn_01x04_Female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

Commit message: finish
Parts:
- removed C8: 100nF, Capacitor_SMD:C_0805_2012Metric
- removed the R24 at (176.0, 114.7)
- removed R48: 10K, Resistor_SMD:R_0805_2012Metric
- removed the TH1 at (176.0, 118.3)
- added ?: MountingHole_3mm, Mounting_Holes:MountingHole_3mm, F.Cu at (53.0, 127.0)
- added ?: MountingHole_3mm, Mounting_Holes:MountingHole_3mm, F.Cu at (103.0, 153.5)
- added G***: LOGO, T0-R0_Stepper_Board:diana, F.Cu at (156.0, 40.5)
- added G***: LOGO, T0-R0_Stepper_Board:diana, F.Cu at (143.5, 104.5)
- added REF**: MountingHole_3mm, Mounting_Holes:MountingHole_3mm, F.Cu at (188.0, 152.0)
- added REF**: MountingHole_3mm, Mounting_Holes:MountingHole_3mm, F.Cu at (188.0, 100.0)
- moved L1 176.5 mm to (70.0, 107.5)
Routing:
- net GNDD: track 446.6 -> 548.9 mm, vias 312 -> 362
- net RST1: track 49.3 -> 104.5 mm, vias 4 -> 6
- net PWMA1: track 17.6 -> 72.0 mm, vias 0 -> 2
- net CW1: track 57.5 -> 110.7 mm, vias 4 -> 7
- net CLK1: track 58.4 -> 110.0 mm, vias 4 -> 5
- net Net-(C23-Pad1): track 16.5 -> 63.3 mm, vias 0 -> 2
- net t_SENS: track 103.1 -> 59.8 mm, vias 3 -> 2
- net Net-(IC1-Pad7): track 63.2 -> 84.7 mm, vias 4 -> 5
- net HALF1: track 77.4 -> 93.2 mm
- net CRTL1: track 79.3 -> 94.9 mm
- net EN1: track 96.6 -> 109.7 mm, vias 3 -> 4
- net +3V3: track 114.4 -> 120.4 mm, vias 12 -> 13
- net PWMB1: track 115.7 -> 119.2 mm, vias 3 -> 4
- net Net-(C8-Pad2): track 17.8 -> 14.8 mm
- net GNDPWR: track 138.0 -> 140.7 mm
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Other:
- outline, holes or cut-outs redrawn
- board text added: "+3v3"
- board text added: "+5V"
- board text added: "A"
- board text added: "ARM STEPPER DRIVER SHOULDER"
- board text added: "B"
- board text added: "E1"
- board text added: "GND"
- board text added: "NRST"
- board text added: "SWCLK"
- board text added: "SWDIO"
- board text added: "TRACESWO"

Commit message: finish2
Routing:
- net +3V3: track 120.4 -> 117.0 mm
Other:
- board text added: "SCL"
- board text added: "SDA"
Changed lines of the file:
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@@
   (general
     (thickness 1.6)
-    (drawings 46)
-    (tracks 1937)
+    (drawings 48)
+    (tracks 1936)
     (zones 0)
     (modules 162)
@@
   )
   (setup
-    (last_trace_width 3)
+    (last_trace_width 0.25)
     (user_trace_width 0.2)
     (user_trace_width 0.4)
@@
       (effects (font (size 1.016 1.016) (thickness 0.254)))
     )
-    (fp_text value L6208D (at 0 0 270) (layer F.SilkS)
+    (fp_text value L6208D (at 0 0 270) (layer F.SilkS) hide
       (effects (font (size 1.016 1.016) (thickness 0.254)))
     )
@@
     (at 40.64 111.76 90)
     (descr "2-way 2.54mm pitch terminal block, Phoenix MPT series")
-    (fp_text reference J5 (at 1.27 -4.50088 90) (layer F.SilkS)
+    (fp_text reference J5 (at 5.26 -1.64 90) (layer F.SilkS)
       (effects (font (size 1 1) (thickness 0.15)))
     )
@@
       (effects (font (size 1.016 1.016) (thickness 0.254)))
     )
-    (fp_text value L6208D (at 0 0 270) (layer F.SilkS)
+    (fp_text value L6208D (at 0 0 270) (layer F.SilkS) hide
       (effects (font (size 1.016 1.016) (thickness 0.254)))
     )
@@
     (descr "Terminal Block Phoenix PT-1,5-2-3.5-H, 2 pins, pitch 3.5mm, size 7x7.6mm^2, drill diamater 1.2mm, pad diameter 2.4mm, see , script-generated using https://github.com/pointhi/kicad-footprint-generator/scripts/TerminalBlock_Phoenix")
     (tags "THT Terminal Block Phoenix PT-1,5-2-3.5-H pitch 3.5mm size 7x7.6mm^2 drill 1.2mm pad 2.4mm")
-    (fp_text reference J1 (at 1.75 -4.16 90) (layer F.SilkS)
+    (fp_text reference J1 (at 2.37 6.09 90) (layer F.SilkS)
       (effects (font (size 1 1) (thickness 0.15)))
     )
@@
     (tags "CMS SOT")
     (attr smd)
-    (fp_text reference U4 (at 0 -4.5 90) (layer F.SilkS)
+    (fp_text reference U4 (at -2.153 4.716 90) (layer F.SilkS)
       (effects (font (size 1 1) (thickness 0.15)))
     )
@@
     (pad 1 np_thru_hole circle (at 0 0) (size 3 3) (drill 3) (layers *.Cu *.Mask))
   )
+  (gr_text SDA (at 45 112 90) (layer F.SilkS)
+    (effects (font (size 1.5 1.5) (thickness 0.3)))
+  )
+  (gr_text SCL (at 45 107.5 90) (layer F.SilkS)
+    (effects (font (size 1.5 1.5) (thickness 0.3)))
+  )
   (gr_poly (pts (xy 167.5 135.5) (xy 167.75 135.5) (xy 167.75 137) (xy 167.5 137)) (layer B.Mask) (width 0.15))
   (gr_poly (pts (xy 162 135.5) (xy 161.5 135.5) (xy 161.5 137) (xy 162 137)) (layer B.Mask) (width 0.15))
@@
   (gr_poly (pts (xy 109.22 110.744) (xy 123.19 110.744) (xy 123.19 117.348) (xy 109.22 117.348)) (layer F.Mask) (width 0.15))
   (gr_poly (pts (xy 109 137) (xy 123 137) (xy 123 144) (xy 109 144)) (layer F.Mask) (width 0.15))
-  (via (at 162.25 118.8) (size 0.8) (drill 0.4) (layers F.Cu B.Cu) (net 56))
-  (via (at 163.4 118.75) (size 0.8) (drill 0.4) (layers F.Cu B.Cu) (net 56))
-  (via (at 164.45 118.8) (size 0.8) (drill 0.4) (layers F.Cu B.Cu) (net 56))
-  (via (at 165.75 118.8) (size 0.8) (drill 0.4) (layers F.Cu B.Cu) (net 56))
-  (via (at 167.05 118.85) (size 0.8) (drill 0.4) (layers F.Cu B.Cu) (net 56))
-  (via (at 167.05 119.85) (size 0.8) (drill 0.4) (layers F.Cu B.Cu) (net 56))
-  (via (at 165.85 119.85) (size 0.8) (drill 0.4) (layers F.Cu B.Cu) (net 56))
-  (via (at 164.55 119.85) (size 0.8) (drill 0.4) (layers F.Cu B.Cu) (net 56))
-  (via (at 163.35 119.8) (size 0.8) (drill 0.4) (layers F.Cu B.Cu) (net 56))
-  (via (at 162.25 119.8) (size 0.8) (drill 0.4) (layers F.Cu B.Cu) (net 56))
   (via (at 186.75 129.25) (size 0.8) (drill 0.4) (layers F.Cu B.Cu) (net 1))
   (via (at 185 126.5) (size 0.8) (drill 0.4) (layers F.Cu B.Cu) (net 1))
@@
   (via (at 80.725 137.275) (size 0.8) (drill 0.4) (layers F.Cu B.Cu) (net 1))
   (via (at 65.175 117.15) (size 0.8) (drill 0.4) (layers F.Cu B.Cu) (net 1))
-  (via (at 110.1852 111.6584) (size 0.8) (drill 0.4) (layers F.Cu B.Cu) (net 56))
   (segment (start 119.953042 105.156) (end 120.0404 105.156) (width 3) (layer F.Cu) (net 1))
   (segment (start 107.014503 105.156) (end 103.610903 108.5596) (width 3) (layer F.Cu) (net 1))
@@
   (segment (start 70.9399 116.43712) (end 70.9399 115.1128) (width 0.2) (layer B.Cu) (net 2))
   (segment (start 67.575 119.80202) (end 70.9399 116.43712) (width 0.2) (layer B.Cu) (net 2))
-  (via (at 68.5125 107.5) (size 0.8) (drill 0.4) (layers F.Cu B.Cu) (net 2))
   (segment (start 67.7625 108.25) (end 68.5125 107.5) (width 0.4) (layer B.Cu) (net 2))
   (segment (start 66.07584 108.25) (end 67.7625 108.25) (width 0.4) (layer B.Cu) (net 2))
@@
   (segment (start 71.4875 107.5) (end 68.5 110.4875) (width 0.4) (layer F.Cu) (net 2))
   (segment (start 68.5 110.67416) (end 68.97624 111.1504) (width 0.4) (layer B.Cu) (net 2))
-  (segment (start 66.07584 108.25) (end 68.5 110.67416) (width 0.4) (layer B.Cu) (net 2))
   (segment (start 74.26452 128.281965) (end 73.52501 129.021475) (width 0.25) (layer F.Cu) (net 2))
   (segment (start 73.52501 129.22499) (end 73.39584 129.35416) (width 0.25) (layer F.Cu) (net 2))
   (segment (start 73.52501 129.021475) (end 73.52501 129.22499) (width 0.25) (layer F.Cu) (net 2))
   (segment (start 74.26452 127.71628) (end 74.26452 128.281965) (width 0.25) (layer F.Cu) (net 2))
+  (via (at 68.5125 107.5) (size 0.8) (drill 0.4) (layers F.Cu B.Cu) (net 2))
   (segment (start 122.8575 126) (end 122.8825 126.025) (width 0.4) (layer F.Cu) (net 3))
   (segment (start 124.5 126) (end 122.8575 126) (width 0.4) (layer F.Cu) (net 3))
@@
   (segment (start 86.651999 126.174999) (end 109.206685 126.174999) (width 0.2) (layer B.Cu) (net 55))
   (segment (start 86.576998 126.25) (end 86.651999 126.174999) (width 0.2) (layer B.Cu) (net 55))
+  (via (at 162.25 118.8) (size 0.8) (drill 0.4) (layers F.Cu B.Cu) (net 56))
+  (via (at 163.4 118.75) (size 0.8) (drill 0.4) (layers F.Cu B.Cu) (net 56))
+  (via (at 164.45 118.8) (size 0.8) (drill 0.4) (layers F.Cu B.Cu) (net 56))
+  (via (at 165.75 118.8) (size 0.8) (drill 0.4) (layers F.Cu B.Cu) (net 56))
+  (via (at 167.05 118.85) (size 0.8) (drill 0.4) (layers F.Cu B.Cu) (net 56))
+  (via (at 167.05 119.85) (size 0.8) (drill 0.4) (layers F.Cu B.Cu) (net 56))
+  (via (at 165.85 119.85) (size 0.8) (drill 0.4) (layers F.Cu B.Cu) (net 56))
+  (via (at 164.55 119.85) (size 0.8) (drill 0.4) (layers F.Cu B.Cu) (net 56))
+  (via (at 163.35 119.8) (size 0.8) (drill 0.4) (layers F.Cu B.Cu) (net 56))
+  (via (at 162.25 119.8) (size 0.8) (drill 0.4) (layers F.Cu B.Cu) (net 56))
+  (via (at 110.1852 111.6584) (size 0.8) (drill 0.4) (layers F.Cu B.Cu) (net 56))
   (via (at 111.1852 111.6584) (size 0.8) (drill 0.4) (layers F.Cu B.Cu) (net 56))
   (via (at 112.1852 111.6584) (size 0.8) (drill 0.4) (layers F.Cu B.Cu) (net 56))

Commit message: finish3
Parts:
- removed C15: 220nF1, Capacitor_SMD:C_0805_2012Metric
- removed C18: 5.6n, Capacitor_SMD:C_0805_2012Metric
- removed C19: 100nF, Capacitor_SMD:C_0805_2012Metric
- removed C20: 10nF, Capacitor_SMD:C_0805_2012Metric
- removed C25: 100nF, Capacitor_SMD:C_1206_3216Metric_Pad1.42x1.75mm_HandSolder
- removed C29: 100uF ceramic, Capacitor_SMD:C_1206_3216Metric_Pad1.42x1.75mm_HandSolder
- removed C32, C33: 1nF, Capacitor_SMD:C_0805_2012Metric
- removed C36, C38: 68nF, Capacitor_SMD:C_0805_2012Metric
- removed D10: LED_RED, LED_SMD:LED_0805_2012Metric
- removed D11, D12, D13, D14: LED, LED_SMD:LED_0805_2012Metric
- removed D4, D6, D8: 1N4148, Diode_SMD:D_SOD-123
- removed IC2: L6208D, T0-R0_Stepper_Board:POWERSO36
- removed J2: M1_CONN, TerminalBlock_Phoenix:TerminalBlock_Phoenix_PT-1,5-4-3.5-H_1x04_P3.50mm_Horizontal
- removed JP5: SolderJumper_2_Bridged, Connector_Wire:SolderWirePad_1x02_P5.08mm_Drill1.5mm
- removed R11: 100, Resistor_SMD:R_0805_2012Metric
- removed R15, R16: 39k, Resistor_SMD:R_0805_2012Metric
- removed R18, R20: 0.3, Resistor_SMD:R_2512_6332Metric
- removed R22: 1k, Resistor_SMD:R_0805_2012Metric
- removed R23, R36: 4.7K, Resistor_SMD:R_0805_2012Metric
- removed R26, R33: 2.2K, Resistor_SMD:R_0805_2012Metric
- removed R37, R38, R39, R40: 10K, Resistor_SMD:R_0805_2012Metric
- removed R9: 100k, Resistor_SMD:R_0805_2012Metric

Commit message: finish4
Parts:
- added SWD: Pin_Header_Straight_1x02_Pitch2.54mm, Pin_Headers:Pin_Header_Straight_1x02_Pitch2.54mm, F.Cu at (72.3, 133.9)
- J10, J11: footprint TerminalBlock_Phoenix:TerminalBlock_Phoenix_MPT-0,5-4-2.54_1x04_P2.54mm_Horizontal -> TerminalBlocks_Phoenix:TerminalBlock_Phoenix_MPT-2.54mm_5pol
- moved SW2 2.50 mm to (97.8, 152.4)
- moved SW3 2.50 mm to (85.0, 152.4)
- moved SW4 2.50 mm to (91.4, 152.4)
- moved SW5 2.50 mm to (78.7, 152.4)
- moved ? 2.40 mm to (105.4, 153.5)
- moved J10 1.84 mm to (51.5, 152.5)
- moved J9 0.71 mm to (40.7, 118.7)
- moved J11 0.25 mm to (65.0, 152.5)
Connections:
- J10 pad 1: +5V -> GNDS
- J10 pad 2: E1_2 -> (no net)
- J10 pad 3: E1_1 -> E1_2
- J10 pad 4: GNDS -> +5V
- J11 pad 1: +5V -> GNDS
- J11 pad 2: E2_2 -> (no net)
- J11 pad 3: E2_1 -> E2_2
- J11 pad 4: GNDS -> +5V
Routing:
- net +12V: track 520.9 -> 530.9 mm
- net USB_DP: track 65.9 -> 71.6 mm
- net I1: track 0.00 -> 5.03 mm
- net I2: track 0.00 -> 4.41 mm
- net E2_1: track 35.6 -> 39.7 mm
- net E1_1: track 45.7 -> 48.1 mm
- net +5V: track 66.8 -> 64.4 mm
- net E3: track 38.3 -> 40.2 mm
- net E2: track 33.2 -> 35.2 mm
- net E4: track 45.1 -> 47.0 mm
- net E1: track 32.0 -> 33.0 mm
- net Net-(J9-Pad1): track 17.1 -> 17.9 mm
- net Net-(J9-Pad3): track 7.86 -> 8.54 mm
- net E2_2: track 38.2 -> 37.5 mm
- net E1_2: track 39.7 -> 40.3 mm
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Other:
- board text added: "12V POWER"
- board text added: "CHARGE PUMP"
- board text added: "GND +"
- board text added: "TX RX"

Commit message: finish 3d
Parts:
- added J1: 12V_CONN, TerminalBlock_Phoenix:TerminalBlock_Phoenix_PT-1,5-2-3.5-H_1x02_P3.50mm_Horizontal, F.Cu at (46.7, 99.4)
- moved J1 3.50 mm to (41.9, 99.4), turned to 270 degrees
- moved J5 3.11 mm to (42.4, 109.2), turned to 270 degrees
Connections:
- J1 pad 1: +12V -> GNDPWR
- J1 pad 2: GNDPWR -> +12V
Routing:
- net i2C1_SCL: track 60.1 -> 58.6 mm
- net i2C1_SDA: track 56.4 -> 55.0 mm
Other:
- board text added: "E2"
- board text added: "E3"
- board text added: "E4"
- board text added: "NC"

Commit message: 4
Parts:
- added C8: 100n, Capacitor_SMD:C_0805_2012Metric, F.Cu at (68.9, 115.7)
- renumbered REF** to M3
Routing:
- net GNDPWR: track 140.7 -> 148.4 mm
- net Net-(C8-Pad2): track 14.8 -> 16.0 mm
- net GNDS: vias 230 -> 218

Commit message: finished
Parts:
- added G***: LOGO, T0-R0_Stepper_Board:logopoli, F.Cu at (141.0, 144.0)
- added R30: 1k, Resistor_SMD:R_0805_2012Metric, F.Cu at (54.2, 110.8)
- added R31: 1k, Resistor_SMD:R_0805_2012Metric, F.Cu at (56.5, 110.5)
Routing:
- net +3V3: track 117.0 -> 121.7 mm
- net i2C1_SDA: track 55.0 -> 56.7 mm, vias 1 -> 2
- net GNDS: vias 218 -> 215
Other:
- board text added: "+3V3"
- board text added: "ARM STEPPER DRIVER SHOULDER REV 1"
- board text added: "GND +12V"
- board text added: "TR_SWO"
- board text removed: "+3v3"
- board text removed: "12V POWER"
- board text removed: "ARM STEPPER DRIVER SHOULDER"
- board text removed: "GND +"
- board text removed: "TRACESWO"

Commit message: gerber
Connections:
- U3 pad 14: Net-(U3-Pad14) -> GNDS
- U3 pad 15: Net-(U3-Pad15) -> GNDS
- U3 pad 20: I3 -> GNDS
- U3 pad 21: I4 -> GNDS
- U3 pad 22: Net-(U3-Pad22) -> GNDS
- U3 pad 26: Net-(U3-Pad26) -> GNDS
- U3 pad 27: Net-(U3-Pad27) -> GNDS
- U3 pad 28: Net-(U3-Pad28) -> GNDS
- U3 pad 29: Net-(U3-Pad29) -> GNDS
- U3 pad 33: FAN1 -> GNDS
- U3 pad 35: Net-(U3-Pad35) -> GNDS
- U3 pad 50: /JTDI -> GNDS
- U3 pad 54: Net-(U3-Pad54) -> GNDS
- U3 pad 56: Net-(U3-Pad56) -> GNDS
Routing:
- net GNDS: track 175.3 -> 192.5 mm, vias 215 -> 218
