File: Arm_stepper.sch (KiCad schematic (older format))
At the start: 125 parts, among them IC1 L6208D, IC2 L6208D, J1 12V_CONN, J10 ENCODER1, J11 ENCODER2, J2 M1_CONN, J3 M1_CONN, J4 Conn_01x06_Male, J5 I2C_CONN, J8 Conn_01x04_Female, J9 USB_B_Mini, M2 Fan, Q2 2N2219, SW1 SW_Push_Dual, SW2 endstop4, SW3 endstop1, SW4 endstop3, SW5 endstop2, U1 ISO1050-00_isolation, U2 USBLC6-2SC6, U3 STM32F446RETx, U4 LM1117-3.3, U5 LM1117-5, Y1 8Mhz

Commit message: init
Parts:
- added JP1: Jumper_NO_Small, Connector_PinSocket_2.54mm:PinSocket_1x02_P2.54mm_Vertical, symbol Device:Jumper_NO_Small
- C1, C10, C11, C12, C13, C14, C15, C17, C18, C19, C2, C20, C23, C24, C26, C27, C28, C3, C30, C32, C33, C34, C35, C36, C38, C4, C5, C7, C8, C9: footprint Capacitors_SMD:C_1206_HandSoldering -> Capacitor_SMD:C_0805_2012Metric
- C21, C22, C25, C29: footprint Capacitors_SMD:C_1206_HandSoldering -> Capacitor_SMD:C_1206_3216Metric_Pad1.42x1.75mm_HandSolder
- D1: footprint Diodes_SMD:D_1206 -> Diode_SMD:D_SOD-123
- D10, D11, D12, D13, D14, D15, D16, D17, D18, D9: footprint LEDs:LED_1206_HandSoldering -> LED_SMD:LED_0805_2012Metric
- D2: footprint LEDs:LED_RGB_1210 -> LED_SMD:LED_RGB_1210
- D4, D5, D6, D8: footprint Diodes_SMD:D_SOD-123 -> Diode_SMD:D_SOD-123
- IC1, IC2: footprint Arm_stepper:POWERSO36 -> T0-R0_Stepper_Board:POWERSO36
- J1: footprint TerminalBlocks_Phoenix:TerminalBlock_Phoenix_PT-3.5mm_2pol -> TerminalBlock_Phoenix:TerminalBlock_Phoenix_PT-1,5-2-3.5-H_1x02_P3.50mm_Horizontal
- J10, J11: footprint TerminalBlocks_Phoenix:TerminalBlock_Phoenix_MPT-2.54mm_4pol -> TerminalBlock_Phoenix:TerminalBlock_Phoenix_MPT-0,5-4-2.54_1x04_P2.54mm_Horizontal
- J2, J3: footprint TerminalBlocks_Phoenix:TerminalBlock_Phoenix_PT-3.5mm_4pol -> TerminalBlock_Phoenix:TerminalBlock_Phoenix_PT-1,5-4-3.5-H_1x04_P3.50mm_Horizontal
- J4: footprint Pin_Headers:Pin_Header_Angled_1x06_Pitch2.54mm -> Connector_PinHeader_2.54mm:PinHeader_1x06_P2.54mm_Vertical
- J5: footprint TerminalBlocks_Phoenix:TerminalBlock_Phoenix_MPT-2.54mm_2pol -> TerminalBlock_Phoenix:TerminalBlock_Phoenix_MPT-0,5-4-2.54_1x04_P2.54mm_Horizontal
- J8: footprint TerminalBlocks_Phoenix:TerminalBlock_Phoenix_MPT-2.54mm_4pol -> Connector_Dsub:DSUB-9_Female_Horizontal_P2.77x2.84mm_EdgePinOffset4.94mm_Housed_MountingHolesOffset7.48mm
- J9: footprint Connectors_USB:USB_Micro-B_Molex-105017-0001 -> Connector_USB:USB_Micro-B_Molex-105017-0001
- JP4, JP5: footprint Wire_Connections_Bridges:WireConnection_1.50mmDrill -> Connector_Wire:SolderWirePad_1x02_P5.08mm_Drill1.5mm
- L1: footprint Inductors_SMD:L_1206_HandSoldering -> Inductor_SMD:L_1206_3216Metric_Pad1.42x1.75mm_HandSolder
- M2: footprint Pin_Headers:Pin_Header_Angled_1x02_Pitch2.54mm -> Connector_PinSocket_2.54mm:PinSocket_1x02_P2.54mm_Vertical
- Q2: footprint TO_SOT_Packages_SMD:SOT-23 -> Package_TO_SOT_SMD:SOT-23_Handsoldering
- R1, R10, R11, R12, R13, R15, R16, R19, R2, R21, R22, R23, R24, R25, R26, R28, R29, R3, R30, R31, R32, R33, R34, R35, R36, R37, R38, R39, R4, R40, R41, R42, R43, R44, R45, R46, R47, R48, R5, R6, R7, R9, TH1: footprint Resistors_SMD:R_1206_HandSoldering -> Resistor_SMD:R_0805_2012Metric
- R14, R17, R18, R20: footprint Resistors_SMD:R_2512_HandSoldering -> Resistor_SMD:R_2512_6332Metric
- SW1: footprint Buttons_Switches_THT:SW_TH_Tactile_Omron_B3F-10xx -> Button_Switch_SMD:SW_SPST_B3S-1000
- SW2, SW3, SW4, SW5: footprint TerminalBlocks_Phoenix:TerminalBlock_Phoenix_MPT-2.54mm_2pol -> TerminalBlock_Phoenix:TerminalBlock_Phoenix_MPT-0,5-2-2.54_1x02_P2.54mm_Horizontal
- U1: footprint ISO1050:SO8 -> Package_SO:SSO-8_6.7x9.8mm_P2.54mm_Clearance8mm
- U2: footprint TO_SOT_Packages_SMD:SOT-23-6_Handsoldering -> Package_TO_SOT_SMD:SOT-23-6_Handsoldering
- U3: footprint Housings_QFP:LQFP-64_10x10mm_Pitch0.5mm -> Package_QFP:LQFP-64_10x10mm_P0.5mm
- U4, U5: footprint TO_SOT_Packages_SMD:SOT-223-3_TabPin2 -> Package_TO_SOT_SMD:SOT-223-3_TabPin2
- Y1: footprint Crystals:Crystal_HC49-U_Vertical -> Crystal:Crystal_HC49-4H_Vertical
Connections:
- net GNDS: now also R33.1
- net at J8.2 (Pin_2), U1.7 (CANH): now also JP1.1; no longer R1.1
- new net: JP1.2, R1.1

Commit message: 4
Parts:
- removed R3: 1k, Resistor_SMD:R_0805_2012Metric, symbol Device:R
- removed R48: 10K, Resistor_SMD:R_0805_2012Metric, symbol Device:R
- added J6: SWDCONNUSART, TerminalBlock_Phoenix:TerminalBlock_Phoenix_MPT-0,5-4-2.54_1x04_P2.54mm_Horizontal, symbol Connector:Conn_01x02_Male
- C15: value 220nF1 -> 220nF Ceramic 50 V
- C20: value 10nF -> 10nF Ceramic 50 V
Connections:
- net +3V3: no longer L1.2, U3.13 (VDDA)
- net at U3.6 (PH1): now also C10.2, Y1.2
- net I1 renamed USART_TX
- net USART_TX: now also J6.1 (Pin_1)
- net I2 renamed USART_RX
- net USART_RX: now also J6.2 (Pin_2)
- new net: L1.2, U3.13 (VDDA)

Commit message: finished
Parts:
- added R30, R31: 10k, Resistor_SMD:R_0805_2012Metric, symbol Device:R
Connections:
- net +3V3: now also R30.2, R31.2
- net i2C1_SCL: now also R31.1
- net i2C1_SDA: now also R30.1
Changed lines of the file:
@@
 Wire Wire Line
 	3600 9950 3800 9950
-Wire Wire Line
-	850  1650 1000 1650
-Wire Wire Line
-	850  1550 1000 1550
 $Comp
 L Connector:Conn_01x02_Male J5
@@
 	1    0    0    -1
 $EndComp
-Text GLabel 1000 1550 2    50   Input ~ 0
+Text GLabel 1950 1550 2    50   Input ~ 0
 i2C1_SDA
-Text GLabel 1000 1650 2    50   Input ~ 0
+Text GLabel 1950 1650 2    50   Input ~ 0
 i2C1_SCL
 $Comp
@@
 P 1050 950
 F 0 "#PWR0107" H 1050 750 50  0001 C CNN
-F 1 "GNDPWR" H 1054 796 50  0000 C CNN
+F 1 "GNDPWR" H 850 800 50  0000 C CNN
 F 2 "" H 1050 900 50  0001 C CNN
 F 3 "" H 1050 900 50  0001 C CNN
@@
 Wire Wire Line
 	3400 3950 4000 3950
+$Comp
+L Device:R R30
+U 1 1 5C853947
+P 1200 1400
+F 0 "R30" V 993 1400 50  0000 C CNN
+F 1 "10k" V 1084 1400 50  0000 C CNN
+F 2 "Resistor_SMD:R_0805_2012Metric" V 1130 1400 50  0001 C CNN
+F 3 "~" H 1200 1400 50  0001 C CNN
+	1    1200 1400
+	-1   0    0    1
+$EndComp
+$Comp
+L Device:R R31
+U 1 1 5C85521B
+P 1550 1300
+F 0 "R31" V 1343 1300 50  0000 C CNN
+F 1 "10k" V 1434 1300 50  0000 C CNN
+F 2 "Resistor_SMD:R_0805_2012Metric" V 1480 1300 50  0001 C CNN
+F 3 "~" H 1550 1300 50  0001 C CNN
+	1    1550 1300
+	-1   0    0    1
+$EndComp
+Wire Wire Line
+	850  1550 1200 1550
+Wire Wire Line
+	1200 1550 1950 1550
+Connection ~ 1200 1550
+Wire Wire Line
+	850  1650 1550 1650
+Wire Wire Line
+	1550 1450 1550 1650
+Connection ~ 1550 1650
+Wire Wire Line
+	1550 1650 1950 1650
+$Comp
+L power:+3.3V #PWR0112
+U 1 1 5C8EB3CB
+P 1200 1250
+F 0 "#PWR0112" H 1200 1100 50  0001 C CNN
+F 1 "+3.3V" H 1215 1423 50  0000 C CNN
+F 2 "" H 1200 1250 50  0001 C CNN
+F 3 "" H 1200 1250 50  0001 C CNN
+	1    1200 1250
+	1    0    0    -1
+$EndComp
+$Comp
+L power:+3.3V #PWR0114
+U 1 1 5C8EBE5F
+P 1550 1150
+F 0 "#PWR0114" H 1550 1000 50  0001 C CNN
+F 1 "+3.3V" H 1565 1323 50  0000 C CNN
+F 2 "" H 1550 1150 50  0001 C CNN
+F 3 "" H 1550 1150 50  0001 C CNN
+	1    1550 1150
+	1    0    0    -1
+$EndComp
 $EndSCHEMATC

Commit message: gerber
Parts:
- removed Q2: 2N2219, Package_TO_SOT_SMD:SOT-23_Handsoldering, symbol Transistor_BJT:2N2219
- added Q?: SQ2364, symbol Device:Q_NMOS_DGS
Connections:
- net GNDPWR: now also Q?.3 (S)
- net at M2.2 (-): now also Q?.1 (D)
- net at R31.2: now also Q?.2 (G)
Other:
- note removed: "Notes:\n1. 3V3 is used as VDD and VDDA for uC. Battery should be disconnected when debugging."
Changed lines of the file:
@@
 Wire Wire Line
 	4900 6000 4900 6300
-Text Notes 3100 7550 0    50   ~ 0
-Notes:\n1. 3V3 is used as VDD and VDDA for uC. Battery should be disconnected when debugging.
 Wire Notes Line
 	3000 6650 3000 7650
@@
 $EndComp
 $Comp
-L Transistor_BJT:2N2219 Q2
-U 1 1 5C30BC3F
-P 14750 8550
-F 0 "Q2" H 14941 8504 50  0000 L CNN
-F 1 "2N2219" H 14941 8595 50  0000 L CNN
-F 2 "Package_TO_SOT_SMD:SOT-23_Handsoldering" H 14950 8475 50  0001 L CIN
-F 3 "http://www.onsemi.com/pub_link/Collateral/2N2219-D.PDF" H 14750 8550 50  0001 L CNN
-	1    14750 8550
-	1    0    0    -1
-$EndComp
-Wire Wire Line
-	14850 8350 14850 8050
-$Comp
 L Device:R R31
 U 1 1 5C3573CB
@@
 	1    0    0    -1
 $EndComp
+$Comp
+L Device:Q_NMOS_DGS Q?
+U 1 1 5C8DEB6F
+P 14750 8550
+F 0 "Q?" H 14955 8596 50  0000 L CNN
+F 1 "SQ2364" H 14955 8505 50  0000 L CNN
+F 2 "" H 14950 8650 50  0001 C CNN
+F 3 "~" H 14750 8550 50  0001 C CNN
+	1    14750 8550
+	1    0    0    -1
+$EndComp
+Wire Wire Line
+	14850 8050 14850 8350
 $EndSCHEMATC
